File: PCB_Salus_II_Prototipo_1/PCB_Salus_II_Prototipo_1.kicad_pcb (KiCad board)
At the start: 2 copper layers, 320 x 205 mm, 43 parts, among them J1 Servo1, J11 Conector Entrada 5V, J12 Conector 5V, J13 Conector Entrada 7V, J14 Conector Salida 7V, J16 Luz2, J17 Cambios1, J18 Cambios 2, J19 MarchaAtras1, J2 Sensor Giro, J20 MarchaAtras2, J21 Sobrante1, J22 Sobrante2, J23 Arranque1, J24 Arranque2, J25 ControlMotor, J3 Acelerador, J4 Conn_01x05_Pin, J5 Servo2, J6 Antena, J7 SensorGiro, J8 Luz1, K1 Rele 5V, K2 Rele 7V, K3 Arranque, Q1 IO25, Q2 IO26, Q3 IO27, Q4 IO14, U1 ESP32-DEVKITC-32D, U2 RASPBERRY_PI_4B_4GB

Commit message: Queda por agregar los ultrasonidos
Parts:
- moved J23 113.2 mm to (69.0, 229.9), turned to 180 degrees
- moved K3 108.1 mm to (77.8, 234.9), turned to 90 degrees
- moved J21 94.1 mm to (140.9, 231.5), turned to 90 degrees
- moved Q4 92.6 mm to (146.0, 225.9), turned to -90 degrees
- moved J22 84.9 mm to (140.9, 225.5), turned to 90 degrees
- moved J19 81.2 mm to (127.0, 231.9), turned to 90 degrees
- moved J8 81.0 mm to (101.0, 232.9), turned to 90 degrees
- moved J17 76.9 mm to (113.9, 232.5), turned to 90 degrees
- moved Q3 74.8 mm to (132.0, 225.9), turned to -90 degrees
- moved J20 70.1 mm to (127.0, 225.9), turned to 90 degrees
- moved J16 67.7 mm to (101.0, 225.9), turned to 90 degrees
- moved Q1 66.6 mm to (107.0, 226.9), turned to -90 degrees
- moved Q2 66.1 mm to (118.9, 226.5), turned to -90 degrees
- moved J18 64.9 mm to (113.9, 226.5), turned to 90 degrees
- moved J24 63.5 mm to (91.0, 216.9), turned to 180 degrees
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Connections:
- Sensor_Corriente1 pad 4: Net-(Driver_Motor1-VIN) -> Net-(Sensor_Corriente1-Cable1)
- Step_7V1 pad 1: Net-(Driver_Motor1-VIN) -> Net-(Sensor_Corriente1-Cable1)
- U1 pad J2-13: unconnected-(U1-IO12-PadJ2-13) -> Acelerador
- U1 pad J3-11: Acelerador -> unconnected-(U1-IO17-PadJ3-11)
Routing:
- net 5V: track 343.5 -> 582.1 mm
- net Corriente: track 469.5 -> 290.2 mm
- net TX ESP: track 128.2 -> 306.1 mm
- net RX ESP: track 88.7 -> 163.3 mm
- net Rele5: track 30.6 -> 37.5 mm
- net Rele4: track 28.8 -> 24.6 mm
- net Rele1: track 18.3 -> 22.4 mm
- net Rele2: track 15.4 -> 19.5 mm
- added copper zone on F.Cu, net GND

Commit message: Modifique la fuente de alimentacion de sensor de Corriente y de giro
Parts:
- moved J7 54.1 mm to (192.0, 184.5)
Connections:
- J1 pad 2: GND -> 7V
- J1 pad 3: 7V -> GND
- J5 pad 2: GND -> 7V
- J5 pad 3: 7V -> GND
- J7 pad 2: 5V -> 3V3
- Sensor_Corriente1 pad 1: 5V -> 3V3
- U1 pad J2-1: unconnected-(U1-3V3-PadJ2-1) -> 3V3
- U1 pad J2-13: Acelerador -> unconnected-(U1-IO12-PadJ2-13)
- U1 pad J3-11: unconnected-(U1-IO17-PadJ3-11) -> Acelerador
Routing:
- net 3V3: track 0.00 -> 357.2 mm
- net 5V: track 582.1 -> 359.5 mm
- net GND: track 459.2 -> 340.7 mm
- net 7V: track 69.7 -> 74.1 mm

Commit message: Se agrego sensores ultrasonidos
Parts:
- added J10: Conn_01x07_Pin, Connector_PinHeader_2.54mm:PinHeader_1x07_P2.54mm_Vertical, F.Cu at (138.6, 151.0)
- added J15: Sensor 1, Connector_PinHeader_2.54mm:PinHeader_1x02_P2.54mm_Vertical, F.Cu at (140.0, 143.5)
- added J26: Sensor 2, Connector_PinHeader_2.54mm:PinHeader_1x02_P2.54mm_Vertical, F.Cu at (159.0, 146.0)
- added J27: Sensor 3, Connector_PinHeader_2.54mm:PinHeader_1x02_P2.54mm_Vertical, F.Cu at (154.0, 146.0)
- added J28: Sensor 4, Connector_PinHeader_2.54mm:PinHeader_1x02_P2.54mm_Vertical, F.Cu at (149.0, 146.0)
- added J29: Sensor 5, Connector_PinHeader_2.54mm:PinHeader_1x02_P2.54mm_Vertical, F.Cu at (145.0, 146.0)
- added J30: Sensor 6, Connector_PinHeader_2.54mm:PinHeader_1x02_P2.54mm_Vertical, F.Cu at (164.0, 146.0)
- added J31: Sensor 7, Connector_PinHeader_2.54mm:PinHeader_1x02_P2.54mm_Vertical, F.Cu at (169.0, 146.0)
- added J9: Conn_01x07_Pin, Connector_PinHeader_2.54mm:PinHeader_1x07_P2.54mm_Vertical, F.Cu at (114.0, 107.1)
- moved J2 47.7 mm to (145.0, 117.0)
- moved J6 17.2 mm to (173.0, 133.0), turned to 90 degrees
- moved J4 3.35 mm to (132.5, 101.0)
- moved J3 3.00 mm to (144.0, 127.0)
Connections:
- U1 pad J2-10: unconnected-(U1-IO26-PadJ2-10) -> Sensor Atras 1
- U1 pad J2-11: unconnected-(U1-IO27-PadJ2-11) -> Sensor Adelante 4
- U1 pad J2-12: unconnected-(U1-IO14-PadJ2-12) -> Sensor Adelante 3
- U1 pad J2-13: unconnected-(U1-IO12-PadJ2-13) -> Sensor Adelante 2
- U1 pad J2-15: unconnected-(U1-IO13-PadJ2-15) -> Sensor Adelante 1
- U1 pad J2-7: SensorGiro -> Corriente
- U1 pad J2-8: Corriente -> Sensor Atras 3
- U1 pad J2-9: unconnected-(U1-IO25-PadJ2-9) -> Sensor Atras 2
- U1 pad J3-10: unconnected-(U1-IO5-PadJ3-10) -> TRIG
- U1 pad J3-16: unconnected-(U1-IO15-PadJ3-16) -> SensorGiro
Routing:
- net L_PWM: track 63.8 -> 86.7 mm
- net Sensor Atras 3: track 0.00 -> 22.8 mm
- net R_PWM: track 64.0 -> 85.6 mm
- net Sensor Atras 2: track 0.00 -> 21.6 mm
- net Sensor Atras 1: track 0.00 -> 21.1 mm
- net Sensor Adelante 4: track 0.00 -> 20.8 mm
- net TRIG: track 0.00 -> 20.2 mm
- net Sensor Adelante 2: track 0.00 -> 20.1 mm
- net Sensor Adelante 3: track 0.00 -> 20.1 mm
- net R_EN_L_EN: track 74.5 -> 94.6 mm
- net Sensor Adelante 1: track 0.00 -> 18.6 mm
- net GND: track 340.7 -> 324.6 mm
- net SensorGiro: track 7.24 -> 20.3 mm
- net 5V: track 359.5 -> 366.9 mm
- net Corriente: track 290.2 -> 294.4 mm
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
Commit message: Se cambio la Ip para configurarlacon WiFi
Parts:
- moved F1 148.0 mm to (234.5, 181.0), turned to 0 degrees
- moved Step_Chino1 92.6 mm to (175.0, 173.0)
- moved Step_7V1 83.7 mm to (187.0, 29.0)
- moved J7 74.6 mm to (130.0, 143.0)
- moved D1 65.4 mm to (177.0, 107.3)
- moved D2 65.4 mm to (161.0, 99.0)
- moved D3 65.4 mm to (79.3, 27.2)
- moved D4 65.4 mm to (68.4, 18.0)
- moved Driver_Motor1 65.4 mm to (126.0, 59.0)
- moved J1 65.4 mm to (39.4, 62.2)
- moved J10 65.4 mm to (86.1, 112.0)
- moved J11 65.4 mm to (195.0, 109.0)
- moved J13 65.4 mm to (94.3, 30.0)
- moved J14 65.4 mm to (35.3, 21.5)
- moved J15 65.4 mm to (87.5, 104.5)
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Routing:
- net Net-(Driver_Motor1-VIN): track 350.1 -> 167.6 mm
- net Net-(Sensor_Corriente1-Cable2): track 9.91 -> 157.6 mm
- net Net-(Sensor_Corriente1-Cable1): track 0.00 -> 63.3 mm
- net GND: track 324.6 -> 301.1 mm
- net Net-(D3-K): track 156.4 -> 135.9 mm
- net 5V: track 366.9 -> 368.6 mm
Other:
- board size 320 x 205 mm -> 293 x 205 mm
