File: Salus III/PCB/PCB_SALUS_III/PCB_SALUS_III.kicad_pcb (KiCad board)
At the start: 2 copper layers, 100 x 100 mm, 53 parts, among them J1 Conn_01x20_Pin, J2 Conn_01x20_Pin, K1 Relay_SPDT, U1 ESP32-DEVKITC-32D

Commit message: Se agrega Word con cosas necesarias para Salus IV
Routing:
- net GND: track 213.3 -> 230.6 mm, vias 29 -> 33
- net Net-(1erTransistor7V1-S): track 34.3 -> 46.8 mm
Changed lines of the file:
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@@
 		(allow_soldermask_bridges_in_footprints no)
 		(pcbplotparams
-			(layerselection 0x00010e0_ffffffff)
+			(layerselection 0x00010f0_ffffffff)
 			(plot_on_all_layers_selection 0x0000000_00000000)
 			(disableapertmacros no)
-			(usegerberextensions no)
-			(usegerberattributes yes)
-			(usegerberadvancedattributes yes)
-			(creategerberjobfile yes)
+			(usegerberextensions yes)
+			(usegerberattributes no)
+			(usegerberadvancedattributes no)
+			(creategerberjobfile no)
 			(dashed_line_dash_ratio 12.000000)
 			(dashed_line_gap_ratio 3.000000)
@@
 			(psa4output no)
 			(plotreference yes)
-			(plotvalue yes)
+			(plotvalue no)
 			(plotfptext yes)
 			(plotinvisibletext no)
 			(sketchpadsonfab no)
-			(subtractmaskfromsilk no)
+			(subtractmaskfromsilk yes)
 			(outputformat 1)
 			(mirror no)
 			(drillshape 0)
 			(scaleselection 1)
-			(outputdirectory "../")
+			(outputdirectory "../Envios/")
 		)
 	)
@@
 		)
 		(fp_text user "${REFERENCE}"
-			(at 0 1.27 360)
+			(at 0 1.27 0)
 			(layer "F.Fab")
 			(effects
@@
 		)
 		(property "Value" "Conn_01x03_Pin"
-			(at 0 7.41 360)
+			(at 0 7.41 0)
 			(layer "F.Fab")
 			(effects
@@
 		)
 		(fp_text user "${REFERENCE}"
-			(at 0 3.81 360)
+			(at 0 3.81 0)
 			(layer "F.Fab")
 			(effects
@@
 		)
 		(fp_text user "${REFERENCE}"
-			(at 0 2.54 360)
+			(at 0 2.54 0)
 			(layer "F.Fab")
 			(effects
@@
 		)
 		(property "Value" "Conn_01x03_Pin"
-			(at 0 7.41 360)
+			(at 0 7.41 0)
 			(layer "F.Fab")
 			(effects
@@
 	)
 	(segment
+		(start 295.2 133.66)
+		(end 307.66 133.66)
+		(width 1)
+		(layer "F.Cu")
+		(net 6)
+	)
+	(segment
 		(start 328.7 128.5)
 		(end 329.48 127.72)
@@
 	)
 	(via
+		(at 247.9 75.1)
+		(size 0.8)
+		(drill 0.3)
+		(layers "F.Cu" "B.Cu")
+		(net 9)
+	)
+	(via
 		(at 316.5 88)
 		(size 0.6)
@@
 	)
 	(via
+		(at 248 81.5)
+		(size 0.8)
+		(drill 0.3)
+		(layers "F.Cu" "B.Cu")
+		(net 9)
+	)
+	(via
 		(at 312.3 121.2)
 		(size 0.8)
@@
 	)
 	(via
+		(at 243.9 99.5)
+		(size 0.8)
+		(drill 0.3)
+		(layers "F.Cu" "B.Cu")
+		(net 9)
+	)
+	(via
 		(at 333.4 97.8)
 		(size 0.8)
@@
 	)
 	(via
+		(at 308.8 51.2)
+		(size 0.8)
+		(drill 0.3)
+		(layers "F.Cu" "B.Cu")
+		(net 9)
+	)
+	(via
 		(at 255.7 119.5)
 		(size 0.8)
@@
 	)
 	(segment
+		(start 242.3 96.9)
+		(end 242 96.9)
+		(width 1)
+		(layer "B.Cu")
+		(net 9)
+	)
+	(segment
+		(start 245.6 74.04)
+		(end 246.36 74.8)
+		(width 1)
+		(layer "B.Cu")
+		(net 9)
+	)
+	(segment
 		(start 316.665 87.835)
 		(end 316.5 88)
@@
 	)
 	(segment
+		(start 308.54 51.470706)
+		(end 308.799998 51.210708)
+		(width 1)
+		(layer "B.Cu")
+		(net 9)
+	)
+	(segment
+		(start 244.84 94.36)
+		(end 242.3 96.9)
+		(width 1)
+		(layer "B.Cu")
+		(net 9)
+	)
+	(segment
+		(start 246.36 74.8)
+		(end 247.6 74.8)
+		(width 1)
+		(layer "B.Cu")
+		(net 9)
+	)
+	(segment
+		(start 242.3 96.9)
+		(end 243.9 98.5)
+		(width 1)
+		(layer "B.Cu")
+		(net 9)
+	)
+	(segment
 		(start 289.8 118.7)
 		(end 289.6 118.5)
@@
 	)
 	(segment
+		(start 247.84 81.66)
+		(end 248 81.5)
+		(width 1)
+		(layer "B.Cu")
+		(net 9)
+	)
+	(segment
+		(start 247.6 74.8)
+		(end 247.9 75.1)
+		(width 1)
+		(layer "B.Cu")
+		(net 9)
+	)
+	(segment
 		(start 300.34 126.76)
 		(end 300.3 126.8)
@@
 	)
 	(segment
+		(start 243.9 98.5)
+		(end 243.9 99.5)
+		(width 1)
+		(layer "B.Cu")
+		(net 9)
+	)
+	(segment
 		(start 300.2 118.7)
 		(end 289.8 118.7)
@@
 	)
 	(segment
+		(start 245.6 99.44)
+		(end 243.96 99.44)
+		(width 1)
+		(layer "B.Cu")
+		(net 9)
+	)
+	(segment
 		(start 286.2 136.8)
 		(end 278 136.8)
@@
 	)
 	(segment
+		(start 245.6 94.36)
+		(end 244.84 94.36)
+		(width 1)
+		(layer "B.Cu")
+		(net 9)
+	)
+	(segment
 		(start 305.3 126.76)
 		(end 300.34 126.76)
 		(width 1)
 		(layer "B.Cu")
+		(net 9)
+	)
+	(segment
+		(start 308.54 53.5)
+		(end 308.54 51.470706)
+		(width 1)
+		(layer "B.Cu")
+		(net 9)
+	)
+	(segment
+		(start 243.96 99.44)
+		(end 243.9 99.5)
+		(width 1)
+		(layer "B.Cu")
+		(net 9)
+	)
+	(segment
+		(start 245.6 81.66)
+		(end 247.84 81.66)
+		(width 1)
+		(layer "B.Cu")
