File: Salus III/PCB/PCB_SALUS_III/_autosave-PCB_SALUS_III.kicad_sch (KiCad schematic)
At the start: 52 parts, among them J1 Conn_01x20_Pin, J2 Conn_01x20_Pin, K1 Relay_SPDT, U1 ESP32-DEVKITC-32D

Commit message: Se agregan algunos cambios
Other:
- note added: "En el diagrama de circuito esta dada vuelta la tira de pinas, eso hay que cambiarlo Y agregar un Pin mas de 5V para que le de la corriente a la Rasp"
- note removed: "En el diagrama de circuito esta dada vuelta la tira de pinas, eso hay que cambiarlo"
Changed lines of the file:
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@@
 		)
 	)
-	(text "En el diagrama de circuito esta dada vuelta la tira de pinas, eso hay que cambiarlo\n"
+	(text "En el diagrama de circuito esta dada vuelta la tira de pinas, eso hay que cambiarlo \nY agregar un Pin mas de 5V para que le de la corriente a la Rasp\n\n"
 		(exclude_from_sim no)
-		(at -34.544 135.382 0)
+		(at -21.336 131.064 0)
 		(effects
 			(font
