File: Salus IV/PCB_SalusIV/Hoja-Base.kicad_pcb (KiCad board)
At the start: 2 copper layers, 100 x 100 mm, 111 parts, among them J3 RC, J4 Pruebas, J5 GPIO1-Libre, J6 GPIO2-Libre, Q1 IRFR5305TRPBF, Q2 IRFR5305TRPBF, Q3 IRFR5305TRPBF, Q4 IRFR5305TRPBF

Commit message: Se agrega terminada antes de modificaciones de mejora
Parts:
- removed JP17, JP18: Jumper_Soldado, Jumper:SolderJumper-2_P1.3mm_Open_Pad1.0x1.5mm
- removed R12, R13, R20, R21, R22, R23, R24, R25, R26, R27, R28, R29, R30, R31, R32, R33, R34: 4.7K, Resistor_SMD:R_1206_3216Metric
- added C9: 100nF, Capacitor_SMD:C_0603_1608Metric, F.Cu at (-1164.2, -115.0)
- added H1: MountingHole, MountingHole:MountingHole_3.2mm_M3, F.Cu at (-1186.2, -39.5)
- added H2: MountingHole, MountingHole:MountingHole_3.2mm_M3, F.Cu at (-1186.2, -131.0)
- added H3: MountingHole, MountingHole:MountingHole_3.2mm_M3, F.Cu at (-1094.9, -130.8)
- added R10: 4.7kΩ, Footprints:RES-ARRAY-SMD_1606-16P-L4.0-W1.6-BL, F.Cu at (-1170.2, -109.5)
- C1, C2, C3, C6, C8: footprint Capacitor_SMD:C_0402_1005Metric -> Capacitor_SMD:C_0603_1608Metric
- C7: footprint Capacitor_SMD:C_0402_1005Metric -> Capacitor_SMD:C_1206_3216Metric
- K1: renamed from Relé-Arranque1; value ~ -> Relé-Arranque
- K2: renamed from Relé-Bateria1; value ~ -> Relé-Bateria
- R18: value 4.7K -> 4.7kΩ; footprint Resistor_SMD:R_1206_3216Metric -> Footprints:RES-ARRAY-SMD_1606-16P-L4.0-W1.6-BL
- U1: renamed from ESP32-S3-WROOM-1-N16; value ~ -> ESP32-S3-WROOM-1-N16
- U2: renamed from TCA9548ARGER1; value ~ -> TCA
- U3: renamed from MCP23017; value ~ -> MCP
- U4: renamed from AMS1117-3.3V1; value ~ -> AMS
- moved Q8 251.9 mm to (-1132.6, -59.9)
- moved J10 251.5 mm to (-1095.6, -119.1), turned to 90 degrees
- moved D3 216.6 mm to (-1135.4, -55.2)
- moved D5 198.8 mm to (-1148.6, -87.6)
- moved J9 198.2 mm to (-1107.2, -40.6)
- moved R11 197.9 mm to (-1131.8, -63.9), turned to -90 degrees
- moved K2 195.9 mm to (-1144.6, -99.8), turned to 90 degrees
- moved R14 194.7 mm to (-1125.9, -116.6)
- moved Q9 192.2 mm to (-1120.2, -96.5), turned to -90 degrees
- moved R37 186.4 mm to (-1123.0, -99.6)
- moved J11 182.8 mm to (-1117.7, -122.3), turned to 180 degrees
- moved R36 173.3 mm to (-1115.0, -105.4)
- moved J14 173.0 mm to (-1123.6, -73.6), turned to -90 degrees
- moved J13 172.2 mm to (-1177.3, -130.6), turned to 180 degrees
- moved J15 163.5 mm to (-1163.9, -125.2)
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- renumbered P3 to J10, TiraEXP1 to J11, Alimentacion-Ultra1 to J12, Acelerador1 to J13, Conectores-Motor1 to J14, Conectores-Carreras1 to J15, Conectores-Giro1 to J16, Conectores-Hall1 to J17, Conectores-Servo1 to J18, TiraMUX1 to J19, Conexiones_Rasp1 to J20, GT-USB-7010ASV1 to J21, 5V1 to J7, 7V1 to J8, Entrada_Logica1 to J9, Reversa1 to Q5, Cambio_Marcha1 to Q6, Luces1 to Q7, Arranque2 to Q8, Arranque1 to Q9
Connections:
- J11 pad 10: Expansor 13 -> Expansor 12
- J11 pad 11: Expansor 6  -> Expansor 5 
- J11 pad 12: Expansor 14 -> Expansor 11
- J11 pad 13: Expansor 7  -> Expansor 4
- J11 pad 14: Expansor 15 -> Expansor 10
- J11 pad 15: Expansor 8 -> Expansor 3
- J11 pad 16: Expansor 16 -> Expansor 9
- J11 pad 2: Expansor 9 -> Expansor 16
- J11 pad 4: Expansor 10 -> Expansor 15
- J11 pad 5: Expansor 3 -> Expansor 8
- J11 pad 6: Expansor 11 -> Expansor 14
- J11 pad 7: Expansor 4 -> Expansor 7 
- J11 pad 8: Expansor 12 -> Expansor 13
- J11 pad 9: Expansor 5  -> Expansor 6 
- J12 pad 10: +5V -> SD2
- J12 pad 12: +5V -> SC2
- J12 pad 14: +5V -> SD3
- J12 pad 16: +5V -> SC3
- J12 pad 2: +5V -> SD4
- J12 pad 4: +5V -> SC4
- J12 pad 6: +5V -> SD1
- J12 pad 8: +5V -> SC1
- J19 pad 1: SD4 -> GND
- J19 pad 10: SD2 -> +5V
- J19 pad 12: SC2 -> +5V
- J19 pad 14: SD3 -> +5V
- J19 pad 16: SC3 -> +5V
- J19 pad 2: GND -> +5V
- J19 pad 3: SC4 -> GND
- J19 pad 4: GND -> +5V
- J19 pad 6: SD1 -> +5V
- J19 pad 8: SC1 -> +5V
- J9 pad 2: Net-(Entrada_Logica1-Pad2) -> Net-(J9-Pad2)
- J9 pad 3: Net-(Cambio_Marcha1-Pad3) -> Net-(J9-Pad3)
- J9 pad 4: Net-(Entrada_Logica1-Pad4) -> Net-(J9-Pad4)
- J9 pad 5: Net-(Entrada_Logica1-Pad5) -> Net-(J9-Pad5)
- K1 pad 2: Net-(Entrada_Logica1-Pad5) -> Net-(J9-Pad2)
- Q5 pad 3: Net-(Entrada_Logica1-Pad4) -> Net-(J9-Pad5)
- Q6 pad 3: Net-(Cambio_Marcha1-Pad3) -> Net-(J9-Pad4)
- Q7 pad 3: Net-(Entrada_Logica1-Pad2) -> Net-(J9-Pad3)
- R16 pad 1: Net-(JP18-B) -> SDA-Expansores
- R16 pad 2: SD0 -> +3.3V
- R17 pad 1: Net-(JP17-B) -> SCL-Expansores
- R17 pad 2: SC0 -> +3.3V
- R18 pad 1: Net-(JP16-B) -> Net-(JP7-B)
- R18 pad 2: SD1 -> Net-(JP6-B)
- R19 pad 1: Net-(JP15-B) -> RST
- R19 pad 2: SC1 -> +3.3V
- U1 pad 20: ENABLE -> RPWM
- U1 pad 22: RPWM -> ENABLE
- U1 pad 4: SDA_Expansor -> SDA-Expansores
- U1 pad 5: SCL_Expansor -> SCL-Expansores
- U1 pad 6: SDA-MUX -> unconnected-(U1-IO6-Pad6)
- U1 pad 7: SCL-MUX -> unconnected-(U1-IO7-Pad7)
- U2 pad 19: SCL-MUX -> SCL-Expansores
- U2 pad 20: SDA-MUX -> SDA-Expansores
- U2 pad 24: RESET -> RST
- U3 pad 12: SCL_Expansor -> SCL-Expansores
- U3 pad 13: SDA_Expansor -> SDA-Expansores
Routing:
- net +3.3V: track 87.8 -> 316.5 mm, vias 5 -> 9
- net GND: track 0.00 -> 164.8 mm, vias 0 -> 82
- net ACELERADOR: track 0.00 -> 161.3 mm, vias 0 -> 2
- net +5V: track 62.7 -> 209.7 mm, vias 2 -> 4
- net Servo2: track 0.00 -> 123.2 mm, vias 0 -> 2
- net SDA-Expansores: track 0.00 -> 121.5 mm, vias 0 -> 8
- net Servo1: track 0.00 -> 119.2 mm, vias 0 -> 3
- net SCL-Expansores: track 0.00 -> 97.4 mm, vias 0 -> 6
- net SD5: track 0.00 -> 80.9 mm, vias 0 -> 3
- net SC5: track 0.00 -> 74.2 mm, vias 0 -> 3
- net 60V: track 0.00 -> 71.2 mm
- net SD6: track 0.00 -> 70.6 mm, vias 0 -> 3
- net RESET: track 16.6 -> 85.4 mm, vias 0 -> 3
- net HALL-1: track 0.00 -> 68.7 mm, vias 0 -> 1
- net HALL-3: track 0.00 -> 68.7 mm, vias 0 -> 1
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- added copper zone on B.Cu, net GND
- added copper zone on F.Cu, net GND
Other:
- outline, holes or cut-outs redrawn

Commit message: Se guarda la PCB Salus IV ya terminada, queda revision final antes de envio
Parts:
- removed D5: 1N6267A, Diode_THT:D_DO-201AE_P15.24mm_Horizontal
- removed the J4 at (-1114.0, -47.4)
- removed the J5 at (-1113.3, -56.6)
- removed the J6 at (-1113.5, -52.1)
- removed K2: Relé-Bateria, Footprints:RELAY-TH_SRD-XXVDC-XL-C
- removed R35: 47K, Footprints:RES-TH_BD2.5-L6.5-P10.50-D0.6
- removed R37: 47K, Resistor_SMD:R_1206_3216Metric
- removed R38, R39: 10K, Resistor_SMD:R_1206_3216Metric
- removed R43: 180, Resistor_SMD:R_1206_3216Metric
- removed R44: 5.1K, Resistor_SMD:R_1206_3216Metric
- added G***: LOGO, Logo:Logo, B.Cu at (-1164.0, -61.3)
- added J17: Pruebas, Connector_PinHeader_2.54mm:PinHeader_1x06_P2.54mm_Vertical, F.Cu at (-1114.0, -47.0)
- added J18: GPIO2-Libre, Connector_PinHeader_2.54mm:PinHeader_1x03_P2.54mm_Vertical, F.Cu at (-1113.3, -52.3)
- added J19: GPIO1-Libre, Connector_PinHeader_2.54mm:PinHeader_1x03_P2.54mm_Vertical, F.Cu at (-1113.4, -56.7)
- added Q10: ~, Footprints:RQ5P0, F.Cu at (-1142.7, -104.1)
- added R12: 47K, Resistor_SMD:R_1206_3216Metric, F.Cu at (-1142.1, -108.8)
- added R13: 1K, Resistor_SMD:R_0603_1608Metric, F.Cu at (-1148.9, -105.6)
- added R20: 47K, Resistor_SMD:R_0603_1608Metric, F.Cu at (-1145.4, -99.7)
- added R21: 47K, Resistor_SMD:R_0603_1608Metric, F.Cu at (-1150.5, -96.8)
- added R22: 10K, Resistor_SMD:R_0603_1608Metric, F.Cu at (-1110.7, -95.0)
- added R23: 10K, Resistor_SMD:R_0603_1608Metric, F.Cu at (-1110.3, -61.3)
- added R24: 180, Resistor_SMD:R_0603_1608Metric, F.Cu at (-1101.7, -56.0)
- added R25: 5.1K, Resistor_SMD:R_0603_1608Metric, F.Cu at (-1103.1, -110.3)
- D3: value 1N6267A -> TPTVS0971P; footprint Diode_THT:D_DO-201AE_P15.24mm_Horizontal -> Footprints:DFN1610-2L_L1.6-W1.0-P1.10-RD
- Q9: value IRLML6344TRPBF -> ~; footprint Footprints:TRANS_IRLML6344TRPBF -> Footprints:SI2301CDS
- R1, R11, R14, R15, R16, R17, R19, R2, R3, R4, R5, R6, R7, R8, R9: footprint Resistor_SMD:R_1206_3216Metric -> Resistor_SMD:R_0603_1608Metric
- R26: renamed from R36; footprint Footprints:RES-TH_BD1.9-L3.3-P7.30-D0.5 -> Resistor_SMD:R_1206_3216Metric
- R27: renamed from R42; footprint Resistor_SMD:R_1206_3216Metric -> Resistor_SMD:R_0603_1608Metric
- R28: renamed from R45; footprint Resistor_SMD:R_1206_3216Metric -> Resistor_SMD:R_0603_1608Metric
- moved Q9 29.1 mm to (-1149.1, -100.1), turned to 0 degrees
- moved R26 27.9 mm to (-1142.1, -98.9), turned to -90 degrees
- moved R17 2.89 mm to (-1133.4, -97.5), turned to 90 degrees
- moved R16 2.87 mm to (-1130.6, -97.5), turned to 90 degrees
- moved R28 1.98 mm to (-1102.9, -106.5)
- moved J16 1.13 mm to (-1097.1, -108.0)
- moved R11 1.09 mm to (-1132.8, -63.5), turned to 90 degrees
- moved R7 0.71 mm to (-1117.9, -63.7), turned to 90 degrees
- moved R4 0.71 mm to (-1185.5, -64.3)
- moved R9 0.50 mm to (-1128.0, -63.5), turned to 90 degrees
- moved R8 0.30 mm to (-1122.2, -63.6), turned to 90 degrees
- moved C7 0.22 mm to (-1101.7, -89.5)
- moved U1 0.15 mm to (-1109.3, -77.0)
- moved R5 0.08 mm to (-1174.7, -51.8), turned to 90 degrees
- moved R6 0.08 mm to (-1170.9, -47.4)
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- renumbered J7 to J1, J13 to J10, J3 to J11, J14 to J12, J19 to J13, J10 to J14, J11 to J15, J21 to J16, J8 to J2, J9 to J3, J20 to J4, J15 to J5, J16 to J6, J17 to J7, J18 to J8, J12 to J9, JP7 to JP1, JP6 to JP2, JP1 to JP3, JP2 to JP4, JP3 to JP5, JP4 to JP6, JP5 to JP7
Connections:
- J13 pad 1: GND -> SD0
- J13 pad 3: GND -> SC0
- Q9 pad 2: GND -> Net-(Q10-G)
- Q9 pad 3: Net-(D5-A1) -> GND
- R11 pad 1: GND -> Arranque
- R11 pad 2: Arranque -> GND
- R16 pad 1: SDA-Expansores -> +3.3V
- R16 pad 2: +3.3V -> SCL-Expansores
- R17 pad 1: SCL-Expansores -> +3.3V
- R17 pad 2: +3.3V -> SDA-Expansores
- R18 pad 10: SDA-Giro -> SD0
- R18 pad 9: SCL-Giro -> SC0
- R5 pad 1: Net-(Q3-G) -> Net-(D2-K)
- R5 pad 2: Net-(D2-K) -> Net-(Q3-G)
- R7 pad 1: GND -> Reversa
- R7 pad 2: Reversa -> GND
- R8 pad 1: GND -> Cambio
- R8 pad 2: Cambio -> GND
- R9 pad 1: GND -> Luces
- R9 pad 2: Luces -> GND
- U1 pad 6: unconnected-(U1-IO6-Pad6) -> SDA-Giro
- U1 pad 7: unconnected-(U1-IO7-Pad7) -> SCL-Giro
- U2 pad 1: SDA-Giro -> SD0
- U2 pad 2: SCL-Giro -> SC0
Routing:
- net SC0: track 0.00 -> 71.7 mm, vias 0 -> 3
- net SD0: track 0.00 -> 53.7 mm, vias 0 -> 4
- net Control_Bat: track 32.4 -> 79.8 mm, vias 2 -> 4
- net SCL-Giro: track 41.0 -> 82.9 mm, vias 3 -> 1
- net SDA-Giro: track 42.5 -> 84.4 mm, vias 2 -> 1
- net Net-(D5-A1): track 36.6 -> 0.00 mm, vias 2 -> 0
- net ADC_ES: track 34.1 -> 59.2 mm, vias 2 -> 4
- net 60V: track 71.2 -> 52.6 mm
- net +5V: track 209.7 -> 224.0 mm
- net Net-(Q10-G): track 0.00 -> 13.3 mm
- net Net-(K2-Pad2): track 5.15 -> 0.00 mm
- net +3.3V: track 316.5 -> 320.5 mm
- net Net-(Q10-D): track 0.00 -> 3.49 mm
- net GND: track 164.8 -> 162.1 mm, vias 82 -> 94
- net TX1: track 52.0 -> 53.8 mm
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